Commit message: Complete S1-M3 simulated sensors

File: src/ai_robot_description/urdf/ai_robot.urdf.xacro (robot description, xacro)
@@ -7,4 +7,12 @@
   <xacro:property name="wheel_width" value="0.035"/>
   <xacro:property name="wheel_y" value="0.18"/>
+  <xacro:property name="laser_samples" value="360"/>
+  <xacro:property name="laser_min_angle" value="-3.14159"/>
+  <xacro:property name="laser_max_angle" value="3.14159"/>
+  <xacro:property name="laser_min_range" value="0.12"/>
+  <xacro:property name="laser_max_range" value="8.0"/>
+  <xacro:property name="camera_width" value="640"/>
+  <xacro:property name="camera_height" value="480"/>
+  <xacro:property name="camera_hfov" value="1.047"/>
   <link name="base_footprint"/>
   <joint name="base_footprint_joint" type="fixed">
@@ -100,3 +108,124 @@
     </plugin>
   </gazebo>
+  <gazebo reference="laser_link">
+    <sensor name="ai_robot_laser" type="ray">
+      <always_on>true</always_on>
+      <visualize>true</visualize>
+      <update_rate>10</update_rate>
+      <ray>
+        <scan>
+          <horizontal>
+            <samples>${laser_samples}</samples>
+            <resolution>1</resolution>
+            <min_angle>${laser_min_angle}</min_angle>
+            <max_angle>${laser_max_angle}</max_angle>
+          </horizontal>
+        </scan>
+        <range>
+          <min>${laser_min_range}</min>
+          <max>${laser_max_range}</max>
+          <resolution>0.01</resolution>
+        </range>
+        <noise>
+          <type>gaussian</type>
+          <mean>0.0</mean>
+          <stddev>0.01</stddev>
+        </noise>
+      </ray>
+      <plugin name="ai_robot_laser_scan" filename="libgazebo_ros_ray_sensor.so">
+        <ros>
+          <remapping>~/out:=/scan</remapping>
+        </ros>
+        <output_type>sensor_msgs/LaserScan</output_type>
+        <frame_name>laser_link</frame_name>
+      </plugin>
+    </sensor>
+  </gazebo>
+  <gazebo reference="camera_link">
+    <sensor name="ai_robot_camera" type="camera">
+      <always_on>true</always_on>
+      <visualize>true</visualize>
+      <update_rate>10</update_rate>
+      <camera>
+        <horizontal_fov>${camera_hfov}</horizontal_fov>
+        <image>
+          <width>${camera_width}</width>
+          <height>${camera_height}</height>
+          <format>R8G8B8</format>
+        </image>
+        <clip>
+          <near>0.05</near>
+          <far>8.0</far>
+        </clip>
+        <noise>
+          <type>gaussian</type>
+          <mean>0.0</mean>
+          <stddev>0.005</stddev>
+        </noise>
+      </camera>
+      <plugin name="ai_robot_camera_driver" filename="libgazebo_ros_camera.so">
+        <ros>
+          <remapping>image_raw:=/camera/image_raw</remapping>
+          <remapping>camera_info:=/camera/camera_info</remapping>
+        </ros>
+        <camera_name>camera</camera_name>
+        <frame_name>camera_link</frame_name>
+      </plugin>
+    </sensor>
+  </gazebo>
+  <gazebo reference="imu_link">
+    <sensor name="ai_robot_imu" type="imu">
+      <always_on>true</always_on>
+      <update_rate>50</update_rate>
+      <imu>
+        <angular_velocity>
+          <x>
+            <noise type="gaussian">
+              <mean>0.0</mean>
+              <stddev>0.0002</stddev>
+            </noise>
+          </x>
+          <y>
+            <noise type="gaussian">
+              <mean>0.0</mean>
+              <stddev>0.0002</stddev>
+            </noise>
+          </y>
+          <z>
+            <noise type="gaussian">
+              <mean>0.0</mean>
+              <stddev>0.0002</stddev>
+            </noise>
+          </z>
+        </angular_velocity>
+        <linear_acceleration>
+          <x>
+            <noise type="gaussian">
+              <mean>0.0</mean>
+              <stddev>0.01</stddev>
+            </noise>
+          </x>
+          <y>
+            <noise type="gaussian">
+              <mean>0.0</mean>
+              <stddev>0.01</stddev>
+            </noise>
+          </y>
+          <z>
+            <noise type="gaussian">
+              <mean>0.0</mean>
+              <stddev>0.01</stddev>
+            </noise>
+          </z>
+        </linear_acceleration>
+      </imu>
+      <plugin name="ai_robot_imu_driver" filename="libgazebo_ros_imu_sensor.so">
+        <ros>
+          <remapping>~/out:=/imu/data</remapping>
+        </ros>
+        <initial_orientation_as_reference>false</initial_orientation_as_reference>
+        <frame_name>imu_link</frame_name>
+      </plugin>
+    </sensor>
+  </gazebo>
 </robot>

Commit message: Fix M2 TF baseline and sync L1 lesson

File: src/ai_robot_description/urdf/ai_robot.urdf.xacro (robot description, xacro)
@@ -30,5 +30,5 @@
       <origin xyz="0 0 ${wheel_radius + body_height / 2}" rpy="0 0 0"/>
       <geometry><box size="${body_length} ${body_width} ${body_height}"/></geometry>
-      <material name="blue"><color rgba="0.1 0.3 0.8 1"/></material>
+      <material name="green"><color rgba="0.1 0.65 0.2 1"/></material>
     </visual>
     <collision>
@@ -81,5 +81,5 @@
     <origin xyz="0 0 ${wheel_radius + body_height}" rpy="0 0 0"/>
   </joint>
-  <gazebo reference="base_link"><material>Gazebo/Blue</material></gazebo>
+  <gazebo reference="base_link"><material>Gazebo/Green</material></gazebo>
   <gazebo reference="left_wheel"><material>Gazebo/Black</material></gazebo>
   <gazebo reference="right_wheel"><material>Gazebo/Black</material></gazebo>
@@ -98,5 +98,5 @@
       <odometry_topic>odom</odometry_topic>
       <odometry_frame>odom</odometry_frame>
-      <robot_base_frame>base_link</robot_base_frame>
+      <robot_base_frame>base_footprint</robot_base_frame>
     </plugin>
   </gazebo>

Commit message: Convert sim base model to four wheels

File: src/ai_robot_description/urdf/ai_robot.urdf.xacro (robot description, xacro)
@@ -6,4 +6,5 @@
   <xacro:property name="wheel_radius" value="0.075"/>
   <xacro:property name="wheel_width" value="0.035"/>
+  <xacro:property name="wheel_x" value="0.16"/>
   <xacro:property name="wheel_y" value="0.18"/>
   <xacro:property name="laser_samples" value="360"/>
@@ -37,5 +38,5 @@
     </collision>
   </link>
-  <xacro:macro name="wheel" params="name y">
+  <xacro:macro name="wheel" params="name x y">
     <link name="${name}">
       <inertial>
@@ -57,10 +58,12 @@
       <parent link="base_link"/>
       <child link="${name}"/>
-      <origin xyz="0 ${y} ${wheel_radius}" rpy="0 0 0"/>
+      <origin xyz="${x} ${y} ${wheel_radius}" rpy="0 0 0"/>
       <axis xyz="0 1 0"/>
     </joint>
   </xacro:macro>
-  <xacro:wheel name="left_wheel" y="${wheel_y}"/>
-  <xacro:wheel name="right_wheel" y="-${wheel_y}"/>
+  <xacro:wheel name="left_front_wheel" x="${wheel_x}" y="${wheel_y}"/>
+  <xacro:wheel name="left_rear_wheel" x="-${wheel_x}" y="${wheel_y}"/>
+  <xacro:wheel name="right_front_wheel" x="${wheel_x}" y="-${wheel_y}"/>
+  <xacro:wheel name="right_rear_wheel" x="-${wheel_x}" y="-${wheel_y}"/>
   <link name="laser_link"/>
   <joint name="laser_joint" type="fixed">
@@ -82,12 +85,19 @@
   </joint>
   <gazebo reference="base_link"><material>Gazebo/Green</material></gazebo>
-  <gazebo reference="left_wheel"><material>Gazebo/Black</material></gazebo>
-  <gazebo reference="right_wheel"><material>Gazebo/Black</material></gazebo>
+  <gazebo reference="left_front_wheel"><material>Gazebo/Black</material></gazebo>
+  <gazebo reference="left_rear_wheel"><material>Gazebo/Black</material></gazebo>
+  <gazebo reference="right_front_wheel"><material>Gazebo/Black</material></gazebo>
+  <gazebo reference="right_rear_wheel"><material>Gazebo/Black</material></gazebo>
   <gazebo>
     <plugin name="ai_robot_diff_drive" filename="libgazebo_ros_diff_drive.so">
       <update_rate>50</update_rate>
-      <left_joint>left_wheel_joint</left_joint>
-      <right_joint>right_wheel_joint</right_joint>
+      <num_wheel_pairs>2</num_wheel_pairs>
+      <left_joint>left_front_wheel_joint</left_joint>
+      <right_joint>right_front_wheel_joint</right_joint>
+      <left_joint>left_rear_wheel_joint</left_joint>
+      <right_joint>right_rear_wheel_joint</right_joint>
       <wheel_separation>0.36</wheel_separation>
+      <wheel_separation>0.36</wheel_separation>
+      <wheel_diameter>0.15</wheel_diameter>
       <wheel_diameter>0.15</wheel_diameter>
       <max_wheel_torque>5.0</max_wheel_torque>
@@ -104,6 +114,8 @@
     <plugin name="ai_robot_joint_states" filename="libgazebo_ros_joint_state_publisher.so">
       <update_rate>50</update_rate>
-      <joint_name>left_wheel_joint</joint_name>
-      <joint_name>right_wheel_joint</joint_name>
+      <joint_name>left_front_wheel_joint</joint_name>
+      <joint_name>left_rear_wheel_joint</joint_name>
+      <joint_name>right_front_wheel_joint</joint_name>
+      <joint_name>right_rear_wheel_joint</joint_name>
     </plugin>
   </gazebo>
