Commit message: 使用SDF显式材质修复小黄车颜色

File: src/ai_robot_description/urdf/small_yellow_car_v1.2.urdf.xacro (robot description, xacro)
@@ -113,5 +113,5 @@
       <origin xyz="0 0 ${wheel_radius + body_height/2}"/>
       <geometry><box size="${body_length} ${body_width} ${body_height}"/></geometry>
-      <material name="Gazebo/Yellow"/>
+      <material name="yellow"/>
     </visual>
     <collision name="body_collision">
